File: hardware/rev0/luna_rev0.kicad_pcb (KiCad board)
At the start: 4 copper layers, 48.9 x 50 mm, 132 parts, among them IC1 ECP5-BGA256, J1 USB_B_Micro, J2 USB_B_Micro, J3 USB_A, J4 USB_B_Micro, J5 Conn_ARM_JTAG_SWD_10, J6 Conn_ARM_JTAG_SWD_10, J7 Conn_02x02_Counter_Clockwise, J8 Conn_Coaxial, J9 Conn_Coaxial, SW1 BTN_RECOVERY, SW2 BTN_DFU, SW3 BTN_RESET, U1 AP22814-SOT, U10 S27KS0641, U11 USB3343, U12 AP22814-SOT, U2 MIC5504-1.8YM5, U3 MIC5219-3.3YM5, U4 TCR2EE11, U5 MIC5504-2.5YM5, U6 ATSAMD21G18A-AUT, U7 W25Q32JVSS, U8 USB3343, U9 USB3343, Y1 DSC60xx

Commit message: Update version and add gerbers
Other:
- board text added: "HACK THE PLANET"
- board text added: "JLCJLCJLCJLCJLC"
- board text added: "r0.2b: May 21th, 2020"
- board text removed: "r0.2: January 26th, 2020"
